File: _autosave-haptic-hands.kicad_pcb (KiCad board)
At the start: 2 copper layers, 67 x 38 mm, 24 parts, among them M1 Motor_DC, SW1 SW_Push, SW2 SW_Push_45deg, SW3 SW_Push_45deg, SW4 SW_Push_45deg, SW5 SW_Push_45deg, SW6 SW_Push_45deg, SW7 SW_Push_45deg, SW8 SW_Push

Commit message: Change schematic & pcb layout again
Routing:
- net (no net): vias 0 -> 1
Changed lines of the file:
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@@
 		(layer "Edge.Cuts")
+	)
+	(via
+		(at 46.9 150.1)
+		(size 6.25)
+		(drill 5.75)
+		(layers "F.Cu" "B.Cu")
+		(net 0)
 	)
 	(segment
