File: _autosave-haptic-hands.kicad_sch (KiCad schematic)
At the start: 24 parts, among them M1 Motor_DC, SW1 SW_Push, SW2 SW_Push_45deg, SW3 SW_Push_45deg, SW4 SW_Push_45deg, SW5 SW_Push_45deg, SW6 SW_Push_45deg, SW7 SW_Push_45deg, SW8 SW_Push

Commit message: Change schematic & pcb layout again
Connections:
- net at C1.1, M1.1 (+): now also SW8.1; no longer SW1.1
- net at SW1.2: no longer SW8.1
- no-connect marks 1 -> 3
Other:
- moved on the sheet: C1, M1, RV1, SW1
