File: haptic-hands.kicad_pcb (KiCad board)
At the start: 2 copper layers, 67 x 38 mm, 24 parts, among them M1 Motor_DC, SW1 SW_Push, SW2 SW_Push_45deg, SW3 SW_Push_45deg, SW4 SW_Push_45deg, SW5 SW_Push_45deg, SW6 SW_Push_45deg, SW7 SW_Push_45deg, SW8 SW_Push

Commit message: Add Haptic Hands logo
Parts:
- added G***: LOGO, LOGO, F.Cu at (76.8, 126.4)
- turned BT1 to 180 degrees
Connections:
- R1 pad 2: Net-(BT1-+) -> Net-(BT1--)
- R2 pad 2: Net-(BT1-+) -> Net-(BT1--)
- R3 pad 2: Net-(BT1-+) -> Net-(BT1--)
- R4 pad 2: Net-(BT1-+) -> Net-(BT1--)
- R5 pad 2: Net-(BT1-+) -> Net-(BT1--)
- R6 pad 2: Net-(BT1-+) -> Net-(BT1--)
- RV1 pad 1: Net-(BT1-+) -> Net-(BT1--)
- SW2 pad 1: Net-(BT1--) -> Net-(BT1-+)
- SW3 pad 1: Net-(BT1--) -> Net-(BT1-+)
- SW4 pad 1: Net-(BT1--) -> Net-(BT1-+)
- SW5 pad 1: Net-(BT1--) -> Net-(BT1-+)
- SW6 pad 1: Net-(BT1--) -> Net-(BT1-+)
- SW7 pad 1: Net-(BT1--) -> Net-(BT1-+)
- SW8 pad 2: Net-(BT1--) -> Net-(BT1-+)
Routing:
- net (no net): vias 0 -> 1
